File: CC26X2R1-hat.kicad_pcb (KiCad board)
At the start: 2 copper layers, 59.7 x 52.3 mm, 11 parts, among them J1 Conn_01x10_Female, J2 Conn_01x10_Female, J3 Conn_01x07, J4 Conn_01x10_Female, J5 Conn_01x10_Female, U1 CC26X2R1

Commit message: Added labels
Parts:
- moved REF** 11.7 mm to (152.1, 93.8)
- moved REF** 9.34 mm to (140.2, 93.2)
Other:
- board text added: "3V3"
- board text added: "GND"
- board text added: "RXD"
- board text added: "TXD"
- board text added: "https://github.com/klein0r/pcb-cc26x2r1-hat"
- board text added: "v0.2"
- board text removed: "v0.1"
Changed lines of the file:
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@@
   (title_block
     (title "CC26X2R1 HAT")
-    (date "2022-01-29")
-    (rev "0.1")
+    (date "2022-02-10")
+    (rev "0.2")
     (company "haus-automatisierung.com")
     (comment 1 "Matthias Kleine")
@@
   (net 43 "unconnected-(J5-Pad4)")
   (footprint "Symbol:WEEE-Logo_4.2x6mm_SilkScreen" (layer "F.Cu")
-    (at 142.875 86.614)
+    (at 152.0634 93.848606)
     (descr "Waste Electrical and Electronic Equipment Directive")
     (tags "Logo WEEE")
@@
     (property "Sheetname" "")
     (attr through_hole)
-    (fp_text reference "U1" (at 0 -0.254 unlocked) (layer "F.SilkS")
+    (fp_text reference "U1" (at 0 5.2324 unlocked) (layer "F.SilkS")
       (effects (font (size 1 1) (thickness 0.15)))
     )
@@
   )
   (footprint "Symbol:KiCad-Logo2_6mm_SilkScreen" (layer "F.Cu")
-    (at 142.875 102.108)
+    (at 140.238514 93.151248)
     (descr "KiCad Logo")
     (tags "Logo KiCad")
@@
     (fp_line (start -1.27 0.635) (end -0.635 1.27) (layer "B.Fab") (width 0.1))
     (fp_line (start 1.27 1.27) (end 1.27 -16.51) (layer "B.Fab") (width 0.1))
-    (pad "1" thru_hole rect (at 0 0 270) (size 1.7 1.7) (drill 1) (layers *.Cu *.Mask)
+    (pad "1" thru_hole oval (at 0 0 270) (size 1.7 1.7) (drill 1) (layers *.Cu *.Mask)
       (net 21 "unconnected-(J3-Pad1)") (pinfunction "Pin_1") (pintype "passive+no_connect"))
     (pad "2" thru_hole oval (at 0 -2.54 270) (size 1.7 1.7) (drill 1) (layers *.Cu *.Mask)
       (net 24 "+3V3") (pinfunction "Pin_2") (pintype "passive"))
-    (pad "3" thru_hole oval (at 0 -5.08 270) (size 1.7 1.7) (drill 1) (layers *.Cu *.Mask)
+    (pad "3" thru_hole rect (at 0 -5.08 270) (size 1.7 1.7) (drill 1) (layers *.Cu *.Mask)
       (net 40 "GND") (pinfunction "Pin_3") (pintype "passive"))
     (pad "4" thru_hole oval (at 0 -7.62 270) (size 1.7 1.7) (drill 1) (layers *.Cu *.Mask)
@@
   (gr_line (start 129.032 60.706) (end 156.718 60.706) (layer "B.SilkS") (width 0.15))
   (gr_line (start 127.762 82.042) (end 127.762 60.96) (layer "Edge.Cuts") (width 0.1))
-  (gr_arc (start 172.72 110.744) (mid 172.348026 111.642025) (end 171.45 112.014) (layer "Edge.Cuts") (width 0.1))
-  (gr_arc (start 159.258 83.312) (mid 158.359975 82.940026) (end 157.988 82.042) (layer "Edge.Cuts") (width 0.1))
-  (gr_arc (start 127.762 60.96) (mid 128.133974 60.061975) (end 129.032 59.69) (layer "Edge.Cuts") (width 0.1))
-  (gr_arc (start 114.3 112.014) (mid 113.401975 111.642026) (end 113.03 110.744) (layer "Edge.Cuts") (width 0.1))
-  (gr_arc (start 171.45 83.312) (mid 172.348025 83.683974) (end 172.72 84.582) (layer "Edge.Cuts") (width 0.1))
+  (gr_arc (start 172.72 110.744) (mid 172.348026 111.642026) (end 171.45 112.014) (layer "Edge.Cuts") (width 0.1))
+  (gr_arc (start 159.258 83.312) (mid 158.359974 82.940026) (end 157.988 82.042) (layer "Edge.Cuts") (width 0.1))
+  (gr_arc (start 127.762 60.96) (mid 128.133974 60.061974) (end 129.032 59.69) (layer "Edge.Cuts") (width 0.1))
+  (gr_arc (start 114.3 112.014) (mid 113.401974 111.642026) (end 113.03 110.744) (layer "Edge.Cuts") (width 0.1))
+  (gr_arc (start 171.45 83.312) (mid 172.348026 83.683974) (end 172.72 84.582) (layer "Edge.Cuts") (width 0.1))
   (gr_line (start 159.258 83.312) (end 171.45 83.312) (layer "Edge.Cuts") (width 0.1))
-  (gr_arc (start 113.03 84.582) (mid 113.401974 83.683975) (end 114.3 83.312) (layer "Edge.Cuts") (width 0.1))
+  (gr_arc (start 113.03 84.582) (mid 113.401974 83.683974) (end 114.3 83.312) (layer "Edge.Cuts") (width 0.1))
   (gr_line (start 129.032 59.69) (end 156.718 59.69) (layer "Edge.Cuts") (width 0.1))
   (gr_line (start 172.72 110.744) (end 172.72 84.582) (layer "Edge.Cuts") (width 0.1))
-  (gr_arc (start 127.762 82.042) (mid 127.390026 82.940025) (end 126.492 83.312) (layer "Edge.Cuts") (width 0.1))
+  (gr_arc (start 127.762 82.042) (mid 127.390026 82.940026) (end 126.492 83.312) (layer "Edge.Cuts") (width 0.1))
   (gr_line (start 114.3 112.014) (end 171.45 112.014) (layer "Edge.Cuts") (width 0.1))
   (gr_line (start 114.3 83.312) (end 126.492 83.312) (layer "Edge.Cuts") (width 0.1))
-  (gr_arc (start 156.718 59.69) (mid 157.616025 60.061974) (end 157.988 60.96) (layer "Edge.Cuts") (width 0.1))
+  (gr_arc (start 156.718 59.69) (mid 157.616026 60.061974) (end 157.988 60.96) (layer "Edge.Cuts") (width 0.1))
   (gr_line (start 157.988 82.042) (end 157.988 60.96) (layer "Edge.Cuts") (width 0.1))
   (gr_line (start 113.03 110.744) (end 113.03 84.582) (layer "Edge.Cuts") (width 0.1))
-  (gr_text "v0.1" (at 155.702 110.236 90) (layer "B.SilkS")
+  (gr_text "https://github.com/klein0r/pcb-cc26x2r1-hat" (at 129.9972 61.214 90) (layer "B.SilkS")
+    (effects (font (size 1 1) (thickness 0.15)) (justify left mirror))
+  )
+  (gr_text "v0.2" (at 155.702 110.236 90) (layer "B.SilkS")
     (effects (font (size 1 1) (thickness 0.15)) (justify right mirror))
   )
@@
     (effects (font (size 2 2) (thickness 0.3)) (justify mirror))
   )
-  (gr_text "This side facing\nbottom of CC26X2R1" (at 142.875 93.472) (layer "F.SilkS")
+  (gr_text "3V3" (at 137.795 107.4 90) (layer "F.SilkS")
+    (effects (font (size 1 1) (thickness 0.15)) (justify left))
+  )
+  (gr_text "RXD" (at 147.955 107.4 90) (layer "F.SilkS")
+    (effects (font (size 1 1) (thickness 0.15)) (justify left))
+  )
+  (gr_text "GND" (at 140.335 107.4 90) (layer "F.SilkS")
+    (effects (font (size 1 1) (thickness 0.15)) (justify left))
+  )
+  (gr_text "This side facing\nbottom of CC26X2R1" (at 142.875 85.5218) (layer "F.SilkS")
     (effects (font (size 1 1) (thickness 0.15)))
   )
+  (gr_text "TXD" (at 145.415 107.4 90) (layer "F.SilkS")
+    (effects (font (size 1 1) (thickness 0.15)) (justify left))
+  )
   (segment (start 116.2 88.9) (end 120.01 88.9) (width 0.25) (layer "B.Cu") (net 1))
   (segment (start 116.2 96.52) (end 120.01 96.52) (width 0.25) (layer "B.Cu") (net 2))
@@
     )
   )
-  (group "" (id 0a358951-dc0f-455f-b40e-a448a2d62296)
-    (members
-      43ade39b-d1cb-4e87-ac4e-a97e95898d50
-      519f6e60-eb9c-479d-80df-fda781585c2a
-      b9f42218-4422-4ebc-a51f-cc675214ea01
-    )
-  )

Commit message: v0.3
Other:
- board text added: "v0.3"
- board text removed: "v0.2"

Commit message: v0.4
Parts:
- removed the G*** at (142.9, 71.9)
- added G***: LOGO, haus-automatisierung:Logo2024, F.Cu at (142.9, 74.9)
- added G***: LOGO, haus-automatisierung:Logo2024, B.Cu at (142.9, 74.9)
- moved REF** 5.00 mm to (152.1, 88.8)
- moved REF** 5.00 mm to (140.2, 88.2)
Other:
- board text added: "Place USR-TCP232-T2 TTL on this side"
- board text added: "v0.4"
- board text removed: "USR-TCP232-T2 TTL"
- board text removed: "haus-automatisierung.com"
- board text removed: "https://github.com/klein0r/pcb-cc26x2r1-hat"
- board text removed: "v0.3"
